Commit message: changed layout of panda to keep consistency

File: panda/urdf/panda.urdf (robot description, URDF)
Before this commit: robot panda, 12 links, 11 joints
Links:
- link panda_hand: geometry collision mesh filename=package://robowflex_resources/panda/meshes/collision/hand.s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; visual mesh filename=package://robowflex_resources/panda/meshes/visual/hand.dae
- link panda_leftfinger: geometry collision mesh filename=package://robowflex_resources/panda/meshes/collision/finger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; visual mesh filename=package://robowflex_resources/panda/meshes/visual/finger.dae
- link panda_link0: geometry collision mesh filename=package://robowflex_resources/panda/meshes/collision/link0.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; visual mesh filename=package://robowflex_resources/panda/meshes/visual/link0.dae
- link panda_link1: geometry collision mesh filename=package://robowflex_resources/panda/meshes/collision/link1.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; visual mesh filename=package://robowflex_resources/panda/meshes/visual/link1.dae
- link panda_link2: geometry collision mesh filename=package://robowflex_resources/panda/meshes/collision/link2.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; visual mesh filename=package://robowflex_resources/panda/meshes/visual/link2.dae
- link panda_link3: geometry collision mesh filename=package://robowflex_resources/panda/meshes/collision/link3.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; visual mesh filename=package://robowflex_resources/panda/meshes/visual/link3.dae
- link panda_link4: geometry collision mesh filename=package://robowflex_resources/panda/meshes/collision/link4.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; visual mesh filename=package://robowflex_resources/panda/meshes/visual/link4.dae
- link panda_link5: geometry collision mesh filename=package://robowflex_resources/panda/meshes/collision/link5.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; visual mesh filename=package://robowflex_resources/panda/meshes/visual/link5.dae
- link panda_link6: geometry collision mesh filename=package://robowflex_resources/panda/meshes/collision/link6.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; visual mesh filename=package://robowflex_resources/panda/meshes/visual/link6.dae
- link panda_link7: geometry collision mesh filename=package://robowflex_resources/panda/meshes/collision/link7.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; visual mesh filename=package://robowflex_resources/panda/meshes/visual/link7.dae
- link panda_rightfinger: geometry collision mesh filename=package://robowflex_resources/panda/meshes/collision/finger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; visual mesh filename=package://robowflex_resources/panda/meshes/visual/finger.dae
