Commit message: Added notable and small table urdf for UR5 and np table srdf

File: ur/robots/ur5_robotiq_robot_limited_notable.urdf.xacro (robot description, xacro)
@@ -1,40 +1,17 @@
 <?xml version="1.0"?>
 <robot xmlns:xacro="http://ros.org/wiki/xacro"
-       name="ur5_robotiq85" >
+       name="ur5_robotiq85_notable" >
   <!-- common stuff -->
-  <xacro:include filename="common.gazebo.xacro" />
+  <xacro:include filename="$(find robowflex_resources)/ur/robots/common.gazebo.xacro" />
   <!-- ur5 -->
-  <xacro:include filename="ur5.urdf.xacro" />
+  <xacro:include filename="$(find robowflex_resources)/ur/robots/ur5.urdf.xacro" />
   <!-- arm -->
-  <xacro:ur5_robot prefix="" joint_limited="true"/>
+  <xacro:ur5_robot prefix="" joint_limited="false"/>
   <link name="world" />
-<!-- box-->
-  <link name="box_link">
-    <visual>
-      <geometry>
-        <box size="0.762 1.524 0.9144"/>
-      </geometry>
-    </visual>
-    <collision>
-      <geometry>
-        <box size="0.762 1.524 0.9144"/>
-      </geometry>
-    </collision>
-    <inertial>
-      <mass value="100"/>
-      <inertia ixx="10" ixy="0.0" ixz="0.0" iyy="10" iyz="0.0" izz="10"/>
-    </inertial>
-  </link>
-<!-- attach the box to the world-->
-  <joint name="world_joint" type="fixed">
-    <parent link="world" />
-    <child link="box_link" />
-    <origin xyz="0.0 0.0 0.4572" rpy="0.0 0.0 0.0" />
-  </joint>
-<!-- attach the robot to the box -->
- <joint name="box_joint" type="fixed">
-    <parent link="box_link"/>
+ <!-- attach the robot to the world -->
+ <joint name="world_joint" type="fixed">
+    <parent link="world"/>
     <child link="base_link"/>
-    <origin xyz="0.0 0.0 0.4572" rpy="0 0 1.57" />
+    <origin xyz="0.5 0.0 0.9184" rpy="0 0 1.57" />
  </joint>
  <!-- Force Torque Sensor -->

File: ur/robots/ur5_robotiq_robot_limited_small.urdf.xacro (robot description, xacro)
@@ -13,10 +13,10 @@
     <visual>
       <geometry>
-        <box size="0.762 1.524 0.9144"/>
+        <box size="0.4 0.4 0.9144"/>
       </geometry>
     </visual>
     <collision>
       <geometry>
-        <box size="0.762 1.524 0.9144"/>
+        <box size="0.4 0.4 0.9144"/>
       </geometry>
     </collision>
