Commit message: Reduced size of table for the UR5 robot

File: ur/robots/ur5_robotiq_robot_limited.urdf.xacro (robot description, xacro)
@@ -10,5 +10,5 @@
   <link name="world" />
 <!-- box-->
-  <link name="box_link">
+  <!--link name="box_link">
     <visual>
       <geometry>
@@ -19,4 +19,21 @@
       <geometry>
         <box size="0.762 1.524 0.9144"/>
+      </geometry>
+    </collision>
+    <inertial>
+      <mass value="100"/>
+      <inertia ixx="10" ixy="0.0" ixz="0.0" iyy="10" iyz="0.0" izz="10"/>
+    </inertial>
+  </link-->
+<!-- box-->
+  <link name="box_link">
+    <visual>
+      <geometry>
+        <box size="0.4 0.4 0.9144"/>
+      </geometry>
+    </visual>
+    <collision>
+      <geometry>
+        <box size="0.4 0.4 0.9144"/>
       </geometry>
     </collision>
@@ -36,5 +53,5 @@
     <parent link="box_link"/>
     <child link="base_link"/>
-    <origin xyz="0.0 -0.381 0.4572" rpy="0 0 1.57" />
+    <origin xyz="0.0 0.0 0.4572" rpy="0 0 1.57" />
  </joint>
  <!-- Force Torque Sensor -->

Commit message: Put back y offset in box_joint for UR5 urdf

File: ur/robots/ur5_robotiq_robot_limited.urdf.xacro (robot description, xacro)
@@ -36,5 +36,5 @@
     <parent link="box_link"/>
     <child link="base_link"/>
-    <origin xyz="0.0 0.0 0.4572" rpy="0 0 1.57" />
+    <origin xyz="0.0 -0.381 0.4572" rpy="0 0 1.57" />
  </joint>
  <!-- Force Torque Sensor -->

Commit message: Correct gripper orientation relative to robot

File: ur/robots/ur5_robotiq_robot_limited.urdf.xacro (robot description, xacro)
@@ -24,5 +24,5 @@
  <xacro:include filename="$(find robowflex_resources)/robotiq/85_gripper/urdf/robotiq_85_gripper.urdf.xacro" />
  <xacro:robotiq_85_gripper prefix="" parent="fts_toolside" >
-   <origin xyz="0.0 0.0 -0.037" rpy="-1.57 3.1415 0.0"/>
+   <origin xyz="0.0 0.0 -0.037" rpy="0.0 0.0 1.57"/>
  </xacro:robotiq_85_gripper>
 </robot>

File: ur/robots/ur5_robotiq_robot_limited_small_table.urdf.xacro (robot description, xacro)
@@ -47,5 +47,5 @@
  <xacro:include filename="$(find robowflex_resources)/robotiq/85_gripper/urdf/robotiq_85_gripper.urdf.xacro" />
  <xacro:robotiq_85_gripper prefix="" parent="fts_toolside" >
-   <origin xyz="0.0 0.0 -0.037" rpy="-1.57 3.1415 0.0"/>
+   <origin xyz="0.0 0.0 -0.037" rpy="0.0 0.0 1.57"/>
  </xacro:robotiq_85_gripper>
 </robot>

File: ur/robots/ur5_robotiq_robot_limited_table.urdf.xacro (robot description, xacro)
@@ -47,5 +47,5 @@
  <xacro:include filename="$(find robowflex_resources)/robotiq/85_gripper/urdf/robotiq_85_gripper.urdf.xacro" />
  <xacro:robotiq_85_gripper prefix="" parent="fts_toolside" >
-   <origin xyz="0.0 0.0 -0.037" rpy="-1.57 3.1415 0.0"/>
+   <origin xyz="0.0 0.0 -0.037" rpy="0.0 0.0 1.57"/>
  </xacro:robotiq_85_gripper>
 </robot>
