Commit message: Made default robot the notable case, and made srdfs xacros

File: ur/config/ur5/ur5_robotiq85.srdf.xacro (robot description, xacro)
@@ -4,5 +4,5 @@
     A URDF file must exist for this robot as well, where the joints and the links that are referenced are defined
 -->
-<robot name="ur5_robotiq85">
+<robot name="ur5_robotiq85" xmlns:xacro="http://www.ros.org/wiki/xacro" >
     <!--GROUPS: Representation of a set of joints and links. This can be useful for specifying DOF to plan for, defining arms, end effectors, etc-->
     <!--LINKS: When a link is specified, the parent joint of that link (if it exists) is automatically included-->
@@ -11,5 +11,5 @@
     <!--SUBGROUPS: Groups can also be formed by referencing to already defined group names-->
     <group name="manipulator">
-        <chain base_link="box_link" tip_link="ee_link" />
+        <chain base_link="base_link" tip_link="ee_link" />
     </group>
     <group name="gripper">
@@ -53,5 +53,5 @@
     <end_effector name="moveit_eef" parent_link="ee_link" group="gripper" />
     <!--VIRTUAL JOINT: Purpose: this element defines a virtual joint between a robot link and an external frame of reference (considered fixed with respect to the robot)-->
-    <virtual_joint name="fixed_joint" type="fixed" parent_frame="world" child_link="box_link" />
+    <!--virtual_joint name="fixed_joint" type="fixed" parent_frame="world" child_link="box_link" /-->
     <!--PASSIVE JOINT: Purpose: this element is used to mark joints that are not actuated-->
     <passive_joint name="robotiq_85_left_finger_tip_joint" />
@@ -61,7 +61,5 @@
     <passive_joint name="robotiq_85_left_inner_knuckle_joint" />
     <!--DISABLE COLLISIONS: By default it is assumed that any link of the robot could potentially come into collision with any other link in the robot. This tag disables collision checking between a specified pair of links. -->
-    <disable_collisions link1="base_link" link2="box_link" reason="Adjacent" />
     <disable_collisions link1="base_link" link2="shoulder_link" reason="Adjacent" />
-    <disable_collisions link1="box_link" link2="shoulder_link" reason="Never" />
     <disable_collisions link1="ee_link" link2="robotiq_85_base_link" reason="Adjacent" />
     <disable_collisions link1="ee_link" link2="robotiq_85_left_finger_link" reason="Never" />

File: ur/robots/ur5_robotiq_robot_limited.urdf.xacro (robot description, xacro)
@@ -3,38 +3,15 @@
        name="ur5_robotiq85" >
   <!-- common stuff -->
-  <xacro:include filename="common.gazebo.xacro" />
+  <xacro:include filename="$(find robowflex_resources)/ur/robots/common.gazebo.xacro" />
   <!-- ur5 -->
-  <xacro:include filename="ur5.urdf.xacro" />
+  <xacro:include filename="$(find robowflex_resources)/ur/robots/ur5.urdf.xacro" />
   <!-- arm -->
-  <xacro:ur5_robot prefix="" joint_limited="true"/>
+  <xacro:ur5_robot prefix="" joint_limited="false"/>
   <link name="world" />
-<!-- box-->
-  <link name="box_link">
-    <visual>
-      <geometry>
-        <box size="0.762 1.524 0.9144"/>
-      </geometry>
-    </visual>
-    <collision>
-      <geometry>
-        <box size="0.762 1.524 0.9144"/>
-      </geometry>
-    </collision>
-    <inertial>
-      <mass value="100"/>
-      <inertia ixx="10" ixy="0.0" ixz="0.0" iyy="10" iyz="0.0" izz="10"/>
-    </inertial>
-  </link>
-<!-- attach the box to the world-->
-  <joint name="world_joint" type="fixed">
-    <parent link="world" />
-    <child link="box_link" />
-    <origin xyz="0.0 0.0 0.4572" rpy="0.0 0.0 0.0" />
-  </joint>
-<!-- attach the robot to the box -->
- <joint name="box_joint" type="fixed">
-    <parent link="box_link"/>
+ <!-- attach the robot to the world -->
+ <joint name="world_joint" type="fixed">
+    <parent link="world"/>
     <child link="base_link"/>
-    <origin xyz="0.0 -0.381 0.4572" rpy="0 0 1.57" />
+    <origin xyz="0.5 0.0 0.9184" rpy="0 0 1.57" />
  </joint>
  <!-- Force Torque Sensor -->

File: ur/robots/ur5_robotiq_robot_limited_table.urdf.xacro (robot description, xacro)
@@ -1,17 +1,40 @@
 <?xml version="1.0"?>
 <robot xmlns:xacro="http://ros.org/wiki/xacro"
-       name="ur5_robotiq85_notable" >
+       name="ur5_robotiq85" >
   <!-- common stuff -->
-  <xacro:include filename="$(find robowflex_resources)/ur/robots/common.gazebo.xacro" />
+  <xacro:include filename="common.gazebo.xacro" />
   <!-- ur5 -->
-  <xacro:include filename="$(find robowflex_resources)/ur/robots/ur5.urdf.xacro" />
+  <xacro:include filename="ur5.urdf.xacro" />
   <!-- arm -->
-  <xacro:ur5_robot prefix="" joint_limited="false"/>
+  <xacro:ur5_robot prefix="" joint_limited="true"/>
   <link name="world" />
- <!-- attach the robot to the world -->
- <joint name="world_joint" type="fixed">
-    <parent link="world"/>
+<!-- box-->
+  <link name="box_link">
+    <visual>
+      <geometry>
+        <box size="0.762 1.524 0.9144"/>
+      </geometry>
+    </visual>
+    <collision>
+      <geometry>
+        <box size="0.762 1.524 0.9144"/>
+      </geometry>
+    </collision>
+    <inertial>
+      <mass value="100"/>
+      <inertia ixx="10" ixy="0.0" ixz="0.0" iyy="10" iyz="0.0" izz="10"/>
+    </inertial>
+  </link>
+<!-- attach the box to the world-->
+  <joint name="world_joint" type="fixed">
+    <parent link="world" />
+    <child link="box_link" />
+    <origin xyz="0.0 0.0 0.4572" rpy="0.0 0.0 0.0" />
+  </joint>
+<!-- attach the robot to the box -->
+ <joint name="box_joint" type="fixed">
+    <parent link="box_link"/>
     <child link="base_link"/>
-    <origin xyz="0.5 0.0 0.9184" rpy="0 0 1.57" />
+    <origin xyz="0.0 -0.381 0.4572" rpy="0 0 1.57" />
  </joint>
  <!-- Force Torque Sensor -->

Commit message: Added UR5 robot descriptions with smaller table and without table (#9)
* Reduced size of table for the UR5 robot

* Added notable and small table urdf for UR5 and np table srdf

* Put back y offset in box_joint for UR5 urdf

* Made default robot the notable case, and made srdfs xacros

* Removed comments, fixed default robot, changed permissions

* Correct gripper orientation relative to robot

Co-authored-by: Constantinos Chamzas <chamzask@gmail.com>
Co-authored-by: Aedan Cullen <aedan@pig.vision>

File: ur/config/ur5/ur5_robotiq85.srdf.xacro (robot description, xacro)
@@ -4,5 +4,5 @@
     A URDF file must exist for this robot as well, where the joints and the links that are referenced are defined
 -->
-<robot name="ur5_robotiq85">
+<robot name="ur5_robotiq85" xmlns:xacro="http://www.ros.org/wiki/xacro" >
     <!--GROUPS: Representation of a set of joints and links. This can be useful for specifying DOF to plan for, defining arms, end effectors, etc-->
     <!--LINKS: When a link is specified, the parent joint of that link (if it exists) is automatically included-->
@@ -11,5 +11,5 @@
     <!--SUBGROUPS: Groups can also be formed by referencing to already defined group names-->
     <group name="manipulator">
-        <chain base_link="box_link" tip_link="ee_link" />
+        <chain base_link="base_link" tip_link="ee_link" />
     </group>
     <group name="gripper">
@@ -52,6 +52,4 @@
     <!--END EFFECTOR: Purpose: Represent information about an end effector.-->
     <end_effector name="moveit_eef" parent_link="ee_link" group="gripper" />
-    <!--VIRTUAL JOINT: Purpose: this element defines a virtual joint between a robot link and an external frame of reference (considered fixed with respect to the robot)-->
-    <virtual_joint name="fixed_joint" type="fixed" parent_frame="world" child_link="box_link" />
     <!--PASSIVE JOINT: Purpose: this element is used to mark joints that are not actuated-->
     <passive_joint name="robotiq_85_left_finger_tip_joint" />
@@ -61,7 +59,5 @@
     <passive_joint name="robotiq_85_left_inner_knuckle_joint" />
     <!--DISABLE COLLISIONS: By default it is assumed that any link of the robot could potentially come into collision with any other link in the robot. This tag disables collision checking between a specified pair of links. -->
-    <disable_collisions link1="base_link" link2="box_link" reason="Adjacent" />
     <disable_collisions link1="base_link" link2="shoulder_link" reason="Adjacent" />
-    <disable_collisions link1="box_link" link2="shoulder_link" reason="Never" />
     <disable_collisions link1="ee_link" link2="robotiq_85_base_link" reason="Adjacent" />
     <disable_collisions link1="ee_link" link2="robotiq_85_left_finger_link" reason="Never" />

File: ur/robots/ur5_robotiq_robot_limited_small_table.urdf.xacro (robot description, xacro)
@@ -3,15 +3,38 @@
        name="ur5_robotiq85" >
   <!-- common stuff -->
-  <xacro:include filename="$(find robowflex_resources)/ur/robots/common.gazebo.xacro" />
+  <xacro:include filename="common.gazebo.xacro" />
   <!-- ur5 -->
-  <xacro:include filename="$(find robowflex_resources)/ur/robots/ur5.urdf.xacro" />
+  <xacro:include filename="ur5.urdf.xacro" />
   <!-- arm -->
   <xacro:ur5_robot prefix="" joint_limited="true"/>
   <link name="world" />
- <!-- attach the robot to the world -->
- <joint name="world_joint" type="fixed">
-    <parent link="world"/>
+<!-- box-->
+  <link name="box_link">
+    <visual>
+      <geometry>
+        <box size="0.4 0.4 0.9144"/>
+      </geometry>
+    </visual>
+    <collision>
+      <geometry>
+        <box size="0.4 0.4 0.9144"/>
+      </geometry>
+    </collision>
+    <inertial>
+      <mass value="100"/>
+      <inertia ixx="10" ixy="0.0" ixz="0.0" iyy="10" iyz="0.0" izz="10"/>
+    </inertial>
+  </link>
+<!-- attach the box to the world-->
+  <joint name="world_joint" type="fixed">
+    <parent link="world" />
+    <child link="box_link" />
+    <origin xyz="0.0 0.0 0.4572" rpy="0.0 0.0 0.0" />
+  </joint>
+<!-- attach the robot to the box -->
+ <joint name="box_joint" type="fixed">
+    <parent link="box_link"/>
     <child link="base_link"/>
-    <origin xyz="0.5 0.0 0.9184" rpy="0 0 1.57" />
+    <origin xyz="0.0 0.0 0.4572" rpy="0 0 1.57" />
  </joint>
  <!-- Force Torque Sensor -->

File: ur/robots/ur5_robotiq_robot_limited_table.urdf.xacro (robot description, xacro)
@@ -3,15 +3,38 @@
        name="ur5_robotiq85" >
   <!-- common stuff -->
-  <xacro:include filename="$(find robowflex_resources)/ur/robots/common.gazebo.xacro" />
+  <xacro:include filename="common.gazebo.xacro" />
   <!-- ur5 -->
-  <xacro:include filename="$(find robowflex_resources)/ur/robots/ur5.urdf.xacro" />
+  <xacro:include filename="ur5.urdf.xacro" />
   <!-- arm -->
   <xacro:ur5_robot prefix="" joint_limited="true"/>
   <link name="world" />
- <!-- attach the robot to the world -->
- <joint name="world_joint" type="fixed">
-    <parent link="world"/>
+<!-- box-->
+  <link name="box_link">
+    <visual>
+      <geometry>
+        <box size="0.762 1.524 0.9144"/>
+      </geometry>
+    </visual>
+    <collision>
+      <geometry>
+        <box size="0.762 1.524 0.9144"/>
+      </geometry>
+    </collision>
+    <inertial>
+      <mass value="100"/>
+      <inertia ixx="10" ixy="0.0" ixz="0.0" iyy="10" iyz="0.0" izz="10"/>
+    </inertial>
+  </link>
+<!-- attach the box to the world-->
+  <joint name="world_joint" type="fixed">
+    <parent link="world" />
+    <child link="box_link" />
+    <origin xyz="0.0 0.0 0.4572" rpy="0.0 0.0 0.0" />
+  </joint>
+<!-- attach the robot to the box -->
+ <joint name="box_joint" type="fixed">
+    <parent link="box_link"/>
     <child link="base_link"/>
-    <origin xyz="0.5 0.0 0.9184" rpy="0 0 1.57" />
+    <origin xyz="0.0 -0.381 0.4572" rpy="0 0 1.57" />
  </joint>
  <!-- Force Torque Sensor -->
